Commit message: Code Modified on Real Robot

File: src/turtlebot_description/urdf/turtlebot_base.xacro (robot description, xacro)
@@ -48,7 +48,8 @@
         </visual>
         <collision>
-            <origin xyz="0.0 0.0 0.0" rpy="0.0 0.0 0.0"/>
+            <origin xyz="0.0 0.0 0.0" rpy="1.57 0.0 0.0"/>
             <geometry>
-                <mesh filename="package://turtlebot_description/meshes/Wheel.stl" scale="0.001 0.001 0.001"/>
+                <cylinder radius="0.039" length="0.021"/>
+                <!-- <mesh filename="package://turtlebot_description/meshes/Wheel.stl" scale="0.001 0.001 0.001"/> -->
             </geometry>
             <material name="black">
@@ -79,7 +80,8 @@
         </visual>
         <collision>
-            <origin xyz="0.0 0.0 0.0" rpy="0.0 0.0 0.0"/>
+            <origin xyz="0.0 0.0 0.0" rpy="1.57 0.0 0.0"/>
             <geometry>
-                <mesh filename="package://turtlebot_description/meshes/Wheel.stl" scale="0.001 0.001 0.001"/>
+                <cylinder radius="0.039" length="0.021"/>
+                <!-- <mesh filename="package://turtlebot_description/meshes/Wheel.stl" scale="0.001 0.001 0.001"/> -->
             </geometry>
             <material name="black">

File: src/turtlebot_description/urdf/turtlebot_ros2control.xacro (robot description, xacro)
@@ -2,7 +2,17 @@
 <robot name="turtlebot" xmlns:xacro="http://www.ros.org/wiki/xacro">
     <ros2_control name="RobotSystem" type="system">
-        <hardware>
-            <plugin>gz_ros2_control/GazeboSimSystem</plugin>
-        </hardware>
+        <!-- ros2_control Gazebo -->
+        <xacro:if value="$(arg is_sim)">
+            <hardware>
+                 <plugin>gz_ros2_control/GazeboSimSystem</plugin>
+            </hardware>
+        </xacro:if>
+        <!-- ros2_control Real Robot -->
+        <xacro:unless value="$(arg is_sim)">
+            <hardware>
+                <plugin>mechabot_firmware/MechabotInterface</plugin>
+                <param name="port">/dev/ttyUSB0</param>
+            </hardware>
+        </xacro:unless>
         <joint name="right_wheel_joint">
             <command_interface name="velocity">

File: src/turtlebot_description/urdf/turtlebot_sensors.xacro (robot description, xacro)
@@ -27,5 +27,5 @@
     </link>
     <joint name="lidar_joint" type="fixed">
-        <origin xyz="-0.003316 0.002508 0.183999" rpy="0.0 0.0 0.0"/>
+        <origin xyz="-0.003316 0.002508 0.183999" rpy="0.0 0.0 3.14159"/>
         <parent link="base_link"/>
         <child link="lidar_link"/>
